File: Opto-Board.kicad_pcb (KiCad board)
At the start: 2 copper layers, 73.7 x 105.4 mm, 62 parts, among them J1 Screw_Terminal_01x08, J2 Screw_Terminal_01x08, J3 Screw_Terminal_01x08, J4 Screw_Terminal_01x02, U1 PC817, U2 PC817, U3 PC817, U4 PC817, U5 PC817, U6 PC817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

Commit message: Some fixes
Parts:
- J1, J2, J3: footprint TerminalBlock_Phoenix:TerminalBlock_Phoenix_MKDS-3-8-5.08_1x08_P5.08mm_Horizontal -> TerminalBlock_Phoenix:TerminalBlock_Phoenix_MKDS-1,5-8_1x08_P5.00mm_Horizontal
- J4: footprint TerminalBlock_Phoenix:TerminalBlock_Phoenix_MKDS-3-2-5.08_1x02_P5.08mm_Horizontal -> TerminalBlock_Phoenix:TerminalBlock_Phoenix_MKDS-1,5-2_1x02_P5.00mm_Horizontal
- moved J2 35.7 mm to (57.8, 115.0), turned to 270 degrees
- moved J3 35.5 mm to (117.4, 110.0), turned to 90 degrees
- moved J1 35.0 mm to (57.8, 75.0), turned to 270 degrees
- moved J4 4.91 mm to (117.4, 126.0), turned to 90 degrees
Connections:
- J1 pad 1: IN5- -> IN8+
- J1 pad 2: IN5+ -> IN8-
- J1 pad 3: IN6- -> IN7+
- J1 pad 4: IN6+ -> IN7-
- J1 pad 5: IN7- -> IN6+
- J1 pad 6: IN7+ -> IN6-
- J1 pad 7: IN8- -> IN5+
- J1 pad 8: IN8+ -> IN5-
- J2 pad 1: IN1- -> IN4+
- J2 pad 2: IN1+ -> IN4-
- J2 pad 3: IN2- -> IN3+
- J2 pad 4: IN2+ -> IN3-
- J2 pad 5: IN3- -> IN2+
- J2 pad 6: IN3+ -> IN2-
- J2 pad 7: IN4- -> IN1+
- J2 pad 8: IN4+ -> IN1-
- J3 pad 1: OUT8 -> OUT1
- J3 pad 2: OUT7 -> OUT2
- J3 pad 3: OUT6 -> OUT3
- J3 pad 4: OUT5 -> OUT4
- J3 pad 5: OUT4 -> OUT5
- J3 pad 6: OUT3 -> OUT6
- J3 pad 7: OUT2 -> OUT7
- J3 pad 8: OUT1 -> OUT8
Routing:
- net IN7-: vias 0 -> 1
- net (no net): vias 4 -> 3

Commit message: More fixes + export
Parts:
- moved R16 1.24 mm to (105.6, 134.9)
- moved R14 1.24 mm to (97.8, 134.9)
Routing:
- net GND2: track 166.9 -> 160.6 mm
- net OUT2: track 58.5 -> 59.7 mm
- net Net-(D8-Pad2): track 3.13 -> 4.25 mm
- net IN7-: vias 1 -> 0
- net (no net): vias 3 -> 4
Other:
- board text added: "INPUT ->"
- board text added: "OUTPUT ->"
- board text removed: "High Voltage"
- board text removed: "Low Voltage"
